Commit message: Simulations for identification

File: urdf/med/med7dock.urdf.xacro (robot description, xacro)
@@ -10,19 +10,11 @@
     <xacro:arg name="sim" default="true" />
     <!-- fix to world -->
-    <link name="world" />
+    <xacro:macro name="extend_link_ee" params="">
     <!-- <link name="world" /> -->
-    <joint name="$(arg robot_name)_joint" type="fixed">
+    <!-- <link name="world" /> -->
+    <!-- <joint name="$(arg robot_name)_joint" type="fixed">
         <parent link="world" />
         <child link="link_0" />
-    </joint>
-    <!-- add med7 robot -->
-    <!-- <xacro:med7 robot_name="$(arg robot_name)" port_id="$(arg port_id)" sim="$(arg sim)" /> -->
-    <!-- <xacro:med7 base_frame="world" robot_name="$(arg robot_name)" sim="$(arg sim)" /> -->
-    <!-- add end-effector -->
-    <joint name="med7_dock_joint" type="fixed">
-        <parent link="link_ee" />
-        <child link="end_effector" />
-        <origin xyz="0 0 0" rpy="0 0 0" />
-    </joint>
+    </joint> -->
     <link name="link_ee">
         <inertial>
@@ -32,4 +24,9 @@
         </inertial>
     </link>
+    <joint name="med7_dock_joint" type="fixed">
+        <parent link="link_ee" />
+        <child link="end_effector" />
+        <origin xyz="0 0 0" rpy="0 0 0" />
+    </joint>
     <link name="end_effector">
     <!-- <inertial>
@@ -59,3 +56,7 @@
     </joint>
     <link name="link_shaft" />
+    </xacro:macro>
+    <!-- <xacro:med7 robot_name="$(arg robot_name)" port_id="$(arg port_id)" sim="$(arg sim)" /> -->
+    <!-- <xacro:med7  robot_name="$(arg robot_name)" sim="$(arg sim)" /> -->
+    <xacro:extend_link_ee/>
 </robot>
